File: 491Project_Darren.kicad_sch (KiCad schematic)
At the start: 49 parts, among them J1 RJ45, J2 RJ45, J3 Conn_01x10_MountingPin

Commit message: changes 0402 footprints to 0805
Parts:
- C1, C10, C13, C14, C15, C16, C2, C5, C6, C7, C8, C9: footprint 491_Footprints:CAP_805_CER -> Capacitor_SMD:C_0805_2012Metric_Pad1.18x1.45mm_HandSolder
- C4: footprint 491_Footprints:CAP_CER_0.1uF_1206 -> Capacitor_SMD:C_0805_2012Metric_Pad1.18x1.45mm_HandSolder
- R1, R10, R11, R12, R13, R14, R15, R16, R17, R18, R19, R2, R20, R21, R23, R24, R3, R4, R5, R6, R7, R8, R9: footprint 491_Footprints:R_805 -> Capacitor_SMD:C_0805_2012Metric_Pad1.18x1.45mm_HandSolder
Changed lines of the file:
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@@
 			)
 		)
-		(property "Footprint" "491_Footprints:R_805"
+		(property "Footprint" "Capacitor_SMD:C_0805_2012Metric_Pad1.18x1.45mm_HandSolder"
 			(at 227.33 113.03 0)
 			(effects
@@
 			)
 		)
-		(property "Footprint" "491_Footprints:CAP_CER_0.1uF_1206"
+		(property "Footprint" "Capacitor_SMD:C_0805_2012Metric_Pad1.18x1.45mm_HandSolder"
 			(at 147.066 79.248 0)
 			(effects
@@
 			)
 		)
-		(property "Footprint" "491_Footprints:R_805"
+		(property "Footprint" "Capacitor_SMD:C_0805_2012Metric_Pad1.18x1.45mm_HandSolder"
 			(at 50.8 171.45 0)
 			(effects
@@
 			)
 		)
-		(property "Footprint" "491_Footprints:R_805"
+		(property "Footprint" "Capacitor_SMD:C_0805_2012Metric_Pad1.18x1.45mm_HandSolder"
 			(at 120.65 163.83 0)
 			(effects
@@
 			)
 		)
-		(property "Footprint" "491_Footprints:R_805"
+		(property "Footprint" "Capacitor_SMD:C_0805_2012Metric_Pad1.18x1.45mm_HandSolder"
 			(at 25.4 85.09 0)
 			(effects
@@
 			)
 		)
-		(property "Footprint" "491_Footprints:R_805"
+		(property "Footprint" "Capacitor_SMD:C_0805_2012Metric_Pad1.18x1.45mm_HandSolder"
 			(at 80.01 194.31 0)
 			(effects
@@
 			)
 		)
-		(property "Footprint" "491_Footprints:R_805"
+		(property "Footprint" "Capacitor_SMD:C_0805_2012Metric_Pad1.18x1.45mm_HandSolder"
 			(at 82.55 139.7 0)
 			(effects
@@
 			)
 		)
-		(property "Footprint" "491_Footprints:CAP_805_CER"
+		(property "Footprint" "Capacitor_SMD:C_0805_2012Metric_Pad1.18x1.45mm_HandSolder"
 			(at 141.986 151.638 0)
 			(effects
@@
 			)
 		)
-		(property "Footprint" "491_Footprints:CAP_805_CER"
+		(property "Footprint" "Capacitor_SMD:C_0805_2012Metric_Pad1.18x1.45mm_HandSolder"
 			(at 122.936 171.958 0)
 			(effects
@@
 			)
 		)
-		(property "Footprint" "491_Footprints:CAP_805_CER"
+		(property "Footprint" "Capacitor_SMD:C_0805_2012Metric_Pad1.18x1.45mm_HandSolder"
 			(at 138.938 40.894 0)
 			(effects
@@
 			)
 		)
-		(property "Footprint" "491_Footprints:CAP_805_CER"
+		(property "Footprint" "Capacitor_SMD:C_0805_2012Metric_Pad1.18x1.45mm_HandSolder"
 			(at 116.586 171.958 0)
 			(effects
@@
 			)
 		)
-		(property "Datasheet" ""
+		(property "Datasheet" "https://www.ti.com/lit/ds/symlink/ths4522.pdf?ts=1712968882721"
 			(at 78.74 162.56 0)
 			(effects
@@
 			)
 		)
-		(property "Footprint" "491_Footprints:R_805"
+		(property "Footprint" "Capacitor_SMD:C_0805_2012Metric_Pad1.18x1.45mm_HandSolder"
 			(at 245.11 113.03 0)
 			(effects
@@
 			)
 		)
-		(property "Footprint" "491_Footprints:R_805"
+		(property "Footprint" "Capacitor_SMD:C_0805_2012Metric_Pad1.18x1.45mm_HandSolder"
 			(at 149.86 186.69 0)
 			(effects
@@
 			)
 		)
-		(property "Footprint" "491_Footprints:R_805"
+		(property "Footprint" "Capacitor_SMD:C_0805_2012Metric_Pad1.18x1.45mm_HandSolder"
 			(at 50.8 162.56 0)
 			(effects
@@
 			)
 		)
-		(property "Footprint" "491_Footprints:R_805"
+		(property "Footprint" "Capacitor_SMD:C_0805_2012Metric_Pad1.18x1.45mm_HandSolder"
 			(at 149.86 195.58 0)
 			(effects
@@
 			)
 		)
-		(property "Datasheet" ""
+		(property "Datasheet" "https://statics.cirrus.com/pubs/proDatasheet/CS8416_DS578F5.pdf"
 			(at 162.56 44.45 0)
 			(effects
@@
 			)
 		)
-		(property "Footprint" "491_Footprints:R_805"
+		(property "Footprint" "Capacitor_SMD:C_0805_2012Metric_Pad1.18x1.45mm_HandSolder"
 			(at 80.01 185.42 0)
 			(effects
@@
 			)
 		)
-		(property "Footprint" "491_Footprints:R_805"
+		(property "Footprint" "Capacitor_SMD:C_0805_2012Metric_Pad1.18x1.45mm_HandSolder"
 			(at 39.37 85.09 0)
 			(effects
@@
 			)
 		)
-		(property "Footprint" "491_Footprints:R_805"
+		(property "Footprint" "Capacitor_SMD:C_0805_2012Metric_Pad1.18x1.45mm_HandSolder"
 			(at 50.8 185.42 0)
 			(effects
@@
 			)
 		)
-		(property "Footprint" "491_Footprints:CAP_805_CER"
+		(property "Footprint" "Capacitor_SMD:C_0805_2012Metric_Pad1.18x1.45mm_HandSolder"
 			(at 74.676 150.368 0)
 			(effects
@@
 			)
 		)
-		(property "Footprint" "491_Footprints:R_805"
+		(property "Footprint" "Capacitor_SMD:C_0805_2012Metric_Pad1.18x1.45mm_HandSolder"
 			(at 121.92 186.69 0)
 			(effects
@@
 			)
 		)
-		(property "Footprint" "491_Footprints:CAP_805_CER"
+		(property "Footprint" "Capacitor_SMD:C_0805_2012Metric_Pad1.18x1.45mm_HandSolder"
 			(at 53.086 169.418 0)
 			(effects
@@
 			)
 		)
-		(property "Footprint" "491_Footprints:CAP_805_CER"
+		(property "Footprint" "Capacitor_SMD:C_0805_2012Metric_Pad1.18x1.45mm_HandSolder"
 			(at 186.436 44.958 0)
 			(effects
@@
 			)
 		)
-		(property "Datasheet" ""
+		(property "Datasheet" "https://www.ti.com/lit/ds/symlink/ths4522.pdf?ts=1712968882721"
 			(at 146.05 163.83 0)
 			(effects
@@
 			)
 		)
-		(property "Footprint" "491_Footprints:CAP_805_CER"
+		(property "Footprint" "Capacitor_SMD:C_0805_2012Metric_Pad1.18x1.45mm_HandSolder"
 			(at 152.146 79.248 0)
 			(effects
@@
 			)
 		)
-		(property "Footprint" "491_Footprints:CAP_805_CER"
+		(property "Footprint" "Capacitor_SMD:C_0805_2012Metric_Pad1.18x1.45mm_HandSolder"
 			(at 171.196 79.248 0)
 			(effects
@@
 			)
 		)
-		(property "Footprint" "491_Footprints:R_805"
+		(property "Footprint" "Capacitor_SMD:C_0805_2012Metric_Pad1.18x1.45mm_HandSolder"
 			(at 167.64 171.45 0)
 			(effects
@@
 			)
 		)
-		(property "Footprint" "491_Footprints:R_805"
+		(property "Footprint" "Capacitor_SMD:C_0805_2012Metric_Pad1.18x1.45mm_HandSolder"
 			(at 167.64 166.37 0)
 			(effects
@@
 			)
 		)
-		(property "Footprint" "491_Footprints:R_805"
+		(property "Footprint" "Capacitor_SMD:C_0805_2012Metric_Pad1.18x1.45mm_HandSolder"
 			(at 149.86 140.97 0)
 			(effects
@@
 			)
 		)
-		(property "Footprint" "491_Footprints:CAP_805_CER"
+		(property "Footprint" "Capacitor_SMD:C_0805_2012Metric_Pad1.18x1.45mm_HandSolder"
 			(at 176.276 88.138 0)
 			(effects
@@
 			)
 		)
-		(property "Footprint" "491_Footprints:R_805"
+		(property "Footprint" "Capacitor_SMD:C_0805_2012Metric_Pad1.18x1.45mm_HandSolder"
 			(at 185.42 58.42 0)
 			(effects
@@
 			)
 		)
-		(property "Footprint" "491_Footprints:R_805"
+		(property "Footprint" "Capacitor_SMD:C_0805_2012Metric_Pad1.18x1.45mm_HandSolder"
 			(at 189.23 80.01 0)
 			(effects
@@
 			)
 		)
-		(property "Footprint" "491_Footprints:CAP_805_CER"
+		(property "Footprint" "Capacitor_SMD:C_0805_2012Metric_Pad1.18x1.45mm_HandSolder"
 			(at 138.938 45.974 0)
 			(effects
@@
 			)
 		)
-		(property "Footprint" "491_Footprints:R_805"
+		(property "Footprint" "Capacitor_SMD:C_0805_2012Metric_Pad1.18x1.45mm_HandSolder"
 			(at 80.01 130.81 0)
 			(effects
@@
 			)
 		)
-		(property "Footprint" "491_Footprints:CAP_805_CER"
+		(property "Footprint" "Capacitor_SMD:C_0805_2012Metric_Pad1.18x1.45mm_HandSolder"
 			(at 58.166 169.418 0)
 			(effects
@@
 			)
 		)
-		(property "Footprint" "491_Footprints:R_805"
+		(property "Footprint" "Capacitor_SMD:C_0805_2012Metric_Pad1.18x1.45mm_HandSolder"
 			(at 129.54 163.83 0)
 			(effects
@@
 			)
 		)
-		(property "Footprint" "491_Footprints:R_805"
+		(property "Footprint" "Capacitor_SMD:C_0805_2012Metric_Pad1.18x1.45mm_HandSolder"
 			(at 50.8 163.83 0)
 			(effects
@@
 			)
 		)
-		(property "Footprint" "491_Footprints:R_805"
+		(property "Footprint" "Capacitor_SMD:C_0805_2012Metric_Pad1.18x1.45mm_HandSolder"
 			(at 149.86 132.08 0)
 			(effects

Commit message: updated silkscreen text to 40 mils
Parts:
- J3: footprint Connector_PinHeader_1.27mm:PinHeader_1x10_P1.27mm_Vertical -> Connector_PinHeader_2.54mm:PinHeader_1x10_P2.54mm_Vertical
Connections:
- net +3V3: now also J3.6 (Pin_6); no longer J3.8 (Pin_8)
- net SIG_IN+: now also J3.10 (Pin_10); no longer J3.7 (Pin_7)
- net SIG_IN-: now also J3.9 (Pin_9); no longer J3.6 (Pin_6)
- net SIG_OUT+: now also J3.8 (Pin_8); no longer J3.10 (Pin_10)
- net SIG_OUT-: now also J3.7 (Pin_7); no longer J3.9 (Pin_9)
Changed lines of the file:
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@@
 	(wire
 		(pts
-			(xy 114.3 29.21) (xy 114.3 40.64)
-		)
-		(stroke
-			(width 0)
-			(type default)
-		)
-	)
-	(wire
-		(pts
 			(xy 71.12 167.64) (xy 68.58 167.64)
 		)
@@
 	(wire
 		(pts
+			(xy 114.3 30.48) (xy 114.3 29.21)
+		)
+		(stroke
+			(width 0)
+			(type default)
+		)
+	)
+	(wire
+		(pts
 			(xy 177.8 58.42) (xy 176.53 58.42)
 		)
@@
 	(wire
 		(pts
-			(xy 109.22 30.48) (xy 109.22 29.21)
+			(xy 109.22 29.21) (xy 109.22 40.64)
 		)
 		(stroke
@@
 		)
 	)
-	(global_label "SIG_IN-"
+	(global_label "SIG_OUT-"
 		(shape input)
-		(at 109.22 30.48 270)
+		(at 111.76 30.48 270)
 		(fields_autoplaced yes)
 		(effects
@@
 		)
 		(property "Intersheetrefs" "${INTERSHEET_REFS}"
-			(at 109.22 38.9155 90)
+			(at 111.76 42.7181 90)
 			(effects
 				(font
@@
 		)
 	)
-	(global_label "AES3-"
-		(shape input)
-		(at 227.33 54.61 180)
-		(fields_autoplaced yes)
-		(effects
-			(font
-				(size 1.016 1.016)
-			)
-			(justify right)
-		)
-		(property "Intersheetrefs" "${INTERSHEET_REFS}"
-			(at 219.9589 54.61 0)
-			(effects
-				(font
-					(size 1.27 1.27)
-				)
-				(justify right)
-				(hide yes)
-			)
-		)
-	)
 	(global_label "PASS+"
 		(shape input)
@@
 		)
 	)
-	(global_label "SIG_OUT+"
+	(global_label "SIG_IN+"
 		(shape input)
-		(at 71.12 26.67 0)
+		(at 119.38 30.48 270)
 		(fields_autoplaced yes)
 		(effects
@@
 				(size 1.016 1.016)
 			)
-			(justify left)
+			(justify right)
 		)
 		(property "Intersheetrefs" "${INTERSHEET_REFS}"
-			(at 83.3581 26.67 0)
+			(at 119.38 38.9155 90)
 			(effects
 				(font
 					(size 1.27 1.27)
 				)
-				(justify left)
+				(justify right)
 				(hide yes)
 			)
 		)
 	)
-	(global_label "FILT"
+	(global_label "SIG_OUT+"
 		(shape input)
-		(at 147.32 45.72 180)
+		(at 71.12 26.67 0)
 		(fields_autoplaced yes)
 		(effects
@@
 				(size 1.016 1.016)
 			)
-			(justify right)
+			(justify left)
 		)
 		(property "Intersheetrefs" "${INTERSHEET_REFS}"
-			(at 141.9808 45.72 0)
+			(at 83.3581 26.67 0)
 			(effects
 				(font
 					(size 1.27 1.27)
 				)
-				(justify right)
+				(justify left)
 				(hide yes)
 			)
 		)
 	)
-	(global_label "SIG_OUT+"
+	(global_label "FILT"
 		(shape input)
-		(at 119.38 30.48 270)
+		(at 147.32 45.72 180)
 		(fields_autoplaced yes)
 		(effects
@@
 		)
 		(property "Intersheetrefs" "${INTERSHEET_REFS}"
-			(at 119.38 42.7181 90)
+			(at 141.9808 45.72 0)
 			(effects
 				(font
@@
 		)
 	)
-	(global_label "SIG_OUT-"
-		(shape input)
-		(at 116.84 30.48 270)
-		(fields_autoplaced yes)
-		(effects
-			(font
-				(size 1.016 1.016)
-			)
-			(justify right)
-		)
-		(property "Intersheetrefs" "${INTERSHEET_REFS}"
-			(at 116.84 42.7181 90)
-			(effects
-				(font
-					(size 1.27 1.27)
-				)
-				(justify right)
-				(hide yes)
-			)
-		)
-	)
 	(global_label "PASS+"
 		(shape input)
@@
 		)
 	)
-	(global_label "AES3+"
-		(shape input)
-		(at 227.33 52.07 180)
-		(fields_autoplaced yes)
-		(effects
-			(font
-				(size 1.016 1.016)
-			)
-			(justify right)
-		)
-		(property "Intersheetrefs" "${INTERSHEET_REFS}"
-			(at 219.9589 52.07 0)
-			(effects
-				(font
-					(size 1.27 1.27)
-				)
-				(justify right)
-				(hide yes)
-			)
-		)
-	)
 	(global_label "FILT"
 		(shape input)
@@
 		)
 	)
+	(global_label "AES3-"
+		(shape input)
+		(at 227.33 54.61 180)
+		(fields_autoplaced yes)
+		(effects
+			(font
+				(size 1.016 1.016)
+			)
+			(justify right)
+		)
+		(property "Intersheetrefs" "${INTERSHEET_REFS}"
+			(at 219.9589 54.61 0)
+			(effects
+				(font
+					(size 1.27 1.27)
+				)
+				(justify right)
+				(hide yes)
+			)
+		)
+	)
 	(global_label "OMCLK"
 		(shape input)
@@
 		)
 	)
-	(global_label "SIG_IN+"
+	(global_label "SIG_IN-"
 		(shape input)
-		(at 111.76 30.48 270)
+		(at 116.84 30.48 270)
 		(fields_autoplaced yes)
 		(effects
@@
 		)
 		(property "Intersheetrefs" "${INTERSHEET_REFS}"
-			(at 111.76 38.9155 90)
+			(at 116.84 38.9155 90)
 			(effects
 				(font
@@
 		)
 	)
+	(global_label "AES3+"
+		(shape input)
+		(at 227.33 52.07 180)
+		(fields_autoplaced yes)
+		(effects
+			(font
+				(size 1.016 1.016)
+			)
+			(justify right)
+		)
+		(property "Intersheetrefs" "${INTERSHEET_REFS}"
+			(at 219.9589 52.07 0)
+			(effects
+				(font
+					(size 1.27 1.27)
+				)
+				(justify right)
+				(hide yes)
+			)
+		)
+	)
 	(global_label "SDA"
 		(shape input)
@@
 		)
 	)
+	(global_label "SIG_OUT+"
+		(shape input)
+		(at 114.3 30.48 270)
+		(fields_autoplaced yes)
+		(effects
+			(font
+				(size 1.016 1.016)
+			)
+			(justify right)
+		)
+		(property "Intersheetrefs" "${INTERSHEET_REFS}"
+			(at 114.3 42.7181 90)
+			(effects
+				(font
+					(size 1.27 1.27)
+				)
+				(justify right)
+				(hide yes)
+			)
+		)
+	)
 	(symbol
 		(lib_id "power:GND")
@@
 	)
 	(symbol
-		(lib_id "power:+3V3")
-		(at 114.3 40.64 0)
-		(mirror x)
-		(unit 1)
-		(exclude_from_sim no)
-		(in_bom yes)
-		(on_board yes)
-		(dnp no)
-		(property "Reference" "#PWR09"
-			(at 114.3 36.83 0)
-			(effects
-				(font
-					(size 1.27 1.27)
-				)
-				(hide yes)
-			)
-		)
-		(property "Value" "+3V3"
-			(at 110.998 44.196 0)
-			(effects
-				(font
-					(size 1.27 1.27)
-				)
-				(justify left)
-			)
-		)
-		(property "Footprint" ""
-			(at 114.3 40.64 0)
-			(effects
-				(font
-					(size 1.27 1.27)
-				)
-				(hide yes)
-			)
-		)
-		(property "Datasheet" ""
-			(at 114.3 40.64 0)
-			(effects
-				(font
-					(size 1.27 1.27)
-				)
-				(hide yes)
-			)
-		)
-		(property "Description" "Power symbol creates a global label with name \"+3V3\""
-			(at 114.3 40.64 0)
-			(effects
-				(font
-					(size 1.27 1.27)
-				)
-				(hide yes)
-			)
-		)
-		(pin "1"
-		)
-		(instances
-			(project "491Project_Darren"
-				(path "/43b85bcc-c949-42f4-ac7f-1cc8aa66ccee"
-					(reference "#PWR09")
-					(unit 1)
-				)
-			)
-		)
-	)
-	(symbol
 		(lib_id "491_Symbols:RES_805")
 		(at 147.32 181.61 0)
@@
 			)
 		)
-		(property "Footprint" "Connector_PinHeader_1.27mm:PinHeader_1x10_P1.27mm_Vertical"
+		(property "Footprint" "Connector_PinHeader_2.54mm:PinHeader_1x10_P2.54mm_Vertical"
 			(at 106.68 24.13 0)
 			(effects
@@
 					(unit 1)
 				)
+			)
+		)
+	)
+	(symbol
+		(lib_id "power:+3V3")
+		(at 109.22 40.64 0)
+		(mirror x)
+		(unit 1)
+		(exclude_from_sim no)
+		(in_bom yes)
+		(on_board yes)
+		(dnp no)
+		(property "Reference" "#PWR09"
+			(at 109.22 36.83 0)
+			(effects
+				(font
+					(size 1.27 1.27)
+				)
+				(hide yes)
+			)
+		)
+		(property "Value" "+3V3"
+			(at 105.918 44.196 0)
+			(effects
+				(font
+					(size 1.27 1.27)
+				)
+				(justify left)
+			)
+		)
+		(property "Footprint" ""
+			(at 109.22 40.64 0)
+			(effects
+				(font
+					(size 1.27 1.27)
+				)
+				(hide yes)
+			)
+		)
+		(property "Datasheet" ""
+			(at 109.22 40.64 0)
+			(effects
+				(font
+					(size 1.27 1.27)
+				)
+				(hide yes)
+			)
+		)
+		(property "Description" "Power symbol creates a global label with name \"+3V3\""
+			(at 109.22 40.64 0)
+			(effects
+				(font
+					(size 1.27 1.27)
+				)
+				(hide yes)
+			)
+		)
+		(pin "1"
+		)
+		(instances
+			(project "491Project_Darren"
+				(path "/43b85bcc-c949-42f4-ac7f-1cc8aa66ccee"
+					(reference "#PWR09")
+					(unit 1)
+				)
